File: corazon leds fade.kicad_pcb (KiCad board)
At the start: 2 copper layers, 79.9 x 77.4 mm, 31 parts, among them J1 Jack-DC, Q1 NMOS, Q2 NMOS, SW1 SW_SPDT, SW2 SW_SPST, U1 NE555P, U2 L78L05_TO92

Commit message: Update corazon leds fade.kicad_pcb
Parts:
- removed C1: C_Polarized, Capacitor_THT:CP_Radial_D5.0mm_P2.00mm
- removed the D1 at (111.8, 67.3)
- removed the D1 at (174.0, 67.3)
- removed D10, D11 (x2), D12, D13 (x2), D14 (x2), D2, D3, D4, D5, D6 (x2), D7 (x2), D8, D9: LED, LED_THT:LED_D4.0mm
- removed J1: Jack-DC, Connector_BarrelJack:BarrelJack_CUI_PJ-102AH_Horizontal
- removed Q1, Q2: NMOS, Package_TO_SOT_THT:TO-220-3_Vertical
- removed R1: R, Resistor_THT:R_Axial_DIN0411_L9.9mm_D3.6mm_P7.62mm_Vertical
- removed RV1, RV2: R_Potentiometer, Potentiometer_THT:Potentiometer_ACP_CA14-H5_Horizontal
- removed SW1: SW_SPDT, Package_TO_SOT_THT:TO-220-3_Vertical
- removed SW2: SW_SPST, Package_TO_SOT_THT:TO-220F-2_Vertical
- removed U1: NE555P, Package_DIP:DIP-8_W7.62mm
- removed U2: L78L05_TO92, Package_TO_SOT_THT:TO-92_Inline
- added D1: D, Diode_THT:D_A-405_P10.16mm_Horizontal, F.Cu at (119.4, 48.3)
- added K1: Relay_SPDT, customFootprints:RELAY_SRD-12VDC-SL-C, F.Cu at (133.0, 42.9)
Routing:
- net Net-(D10-A): track 166.4 -> 0.00 mm
- net Net-(D1-A): track 141.9 -> 0.00 mm
- net Net-(U1-R): track 91.3 -> 0.00 mm
- net Net-(D12-K): track 80.1 -> 0.00 mm
- net Net-(D4-K): track 56.7 -> 0.00 mm
- net Net-(D1-K): track 50.1 -> 0.00 mm
- net Net-(D11-K): track 41.4 -> 0.00 mm
- net Net-(SW2-A): track 26.0 -> 0.00 mm
- net Net-(D3-K): track 25.1 -> 0.00 mm
- net Net-(U2-VI): track 23.2 -> 0.00 mm
- net Net-(C1-Pad2): track 15.1 -> 0.00 mm
- net Net-(SW2-B): track 10.8 -> 0.00 mm
- net (no net): vias 1 -> 0
Other:
- board outline removed

Commit message: Update corazon leds fade.kicad_pcb
Parts:
- removed K1: Relay_SPDT, customFootprints:RELAY_SRD-12VDC-SL-C
- added C1: C_Polarized, Capacitor_THT:CP_Radial_D5.0mm_P2.00mm, B.Cu at (205.8, 95.2)
- added D10: LED, LED_THT:LED_D4.0mm, F.Cu at (197.0, 91.2)
- added D11: LED, LED_THT:LED_D4.0mm, F.Cu at (138.8, 72.4)
- added D12: LED, LED_THT:LED_D4.0mm, F.Cu at (145.3, 72.4)
- added D13: LED, LED_THT:LED_D4.0mm, F.Cu at (184.0, 97.8)
- added D14: LED, LED_THT:LED_D4.0mm, F.Cu at (190.5, 97.8)
- added D2: LED, LED_THT:LED_D4.0mm, F.Cu at (145.3, 63.5)
- added D3: LED, LED_THT:LED_D4.0mm, F.Cu at (151.8, 63.5)
- added D4: LED, LED_THT:LED_D4.0mm, F.Cu at (158.3, 63.5)
- added D5: LED, LED_THT:LED_D4.0mm, F.Cu at (164.8, 63.5)
- added D6: LED, LED_THT:LED_D4.0mm, F.Cu at (171.0, 91.2)
- added D7: LED, LED_THT:LED_D4.0mm, F.Cu at (177.5, 91.2)
- added D8: LED, LED_THT:LED_D4.0mm, F.Cu at (184.0, 91.2)
- added D9: LED, LED_THT:LED_D4.0mm, F.Cu at (190.5, 91.2)
- added J1: Jack-DC, Connector_BarrelJack:BarrelJack_CUI_PJ-102AH_Horizontal, B.Cu at (192.4, 103.4)
- added Q1: NMOS, Package_TO_SOT_THT:TO-220-3_Vertical, B.Cu at (142.9, 89.8)
- added Q2: NMOS, Package_TO_SOT_THT:TO-220-3_Vertical, B.Cu at (193.0, 76.5)
- added R1: R, Resistor_THT:R_Axial_DIN0411_L9.9mm_D3.6mm_P7.62mm_Vertical, B.Cu at (189.5, 120.7)
- added RV1: R_Potentiometer, Potentiometer_THT:Potentiometer_ACP_CA14-H5_Horizontal, B.Cu at (175.3, 117.5)
- added RV2: R_Potentiometer, Potentiometer_THT:Potentiometer_ACP_CA14-H5_Horizontal, B.Cu at (159.3, 128.3)
- added SW2: SW_SPST, Package_TO_SOT_THT:TO-220F-2_Vertical, B.Cu at (207.6, 117.5)
- added U1: NE555P, Package_DIP:DIP-8_W7.62mm, B.Cu at (215.9, 83.2)
- added U2: L78L05_TO92, Package_TO_SOT_THT:TO-92_Inline, B.Cu at (171.0, 119.9)
- D1: value D -> LED; footprint Diode_THT:D_A-405_P10.16mm_Horizontal -> LED_THT:LED_D4.0mm
- moved D1 25.0 mm to (139.2, 63.5), turned to 0 degrees
Other:
- board outline added: 79.8 x 77.4 mm

Commit message: Update corazon leds fade.kicad_pcb
Parts:
- added D15: LED, LED_THT:LED_D4.0mm, F.Cu at (168.3, 44.5)
- added D16: LED, LED_THT:LED_D4.0mm, F.Cu at (156.8, 50.8)
- moved J1 83.4 mm to (119.4, 63.1), turned to 0 degrees
- moved SW2 77.2 mm to (158.7, 57.9), turned to -90 degrees
- moved U2 70.9 mm to (131.8, 60.8)
- moved RV2 65.3 mm to (130.3, 69.8)
- moved R1 61.5 mm to (173.7, 61.3), turned to -90 degrees
- moved D5 56.8 mm to (107.9, 62.3)
- moved U1 56.2 mm to (170.9, 49.5)
- moved C1 52.1 mm to (165.6, 62.2)
- moved D4 51.3 mm to (108.6, 50.8)
- moved D14 48.2 mm to (179.7, 50.8), turned to 180 degrees
- moved Q2 46.6 mm to (148.4, 63.0), turned to 90 degrees
- moved RV1 41.3 mm to (158.0, 79.9)
- moved D6 38.6 mm to (132.7, 96.4)
- moved D7 38.4 mm to (142.9, 107.9)
- moved D3 37.0 mm to (120.0, 44.6)
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Other:
- board text added: "BATTERY"
- board text added: "FALTA PORTAPILAS 9V"
